File: hardware/PCB design/WPS_Scaled/User_Interface.kicad_sch (KiCad schematic)
At the start: 11 parts, among them J13 ZX-XH2.54-2PZZ, J14 2.54-1*4P母, J15 ZX-XH2.54-2PZZ, J16 ZX-XH2.54-2PZZ

Commit message: finallized pcb layout
Parts:
- removed R33, R34: 4.7k, symbol Device:R
- C19: footprint (none) -> COIL:CAP-TH_L3.6-W2.3-P2.50-D0.5
- J13, J15, J16: footprint :CONN-TH_2P-P2.50_HX25003-2A -> COIL:CONN-TH_2P-P2.50_HX25003-2A
- J14: footprint :HDR-TH_4P-P2.54-V-F -> COIL:HDR-TH_4P-P2.54-V-F
- R22, R23, R24, R25: footprint (none) -> COIL:RES-TH_BD2.4-L6.3-P10.30-D0.6
Connections:
- net BUTTON_P: now reaches J13.1, R22.2, R23.1
- net LED_MAINTENANCE_P: now reaches J16.1, R25.1
- net LED_POWER_P: now reaches J15.1, R24.1
- net +3.3V renamed +3V3
Other:
- moved on the sheet: J13, J14, J15, J16
