File: hardware/PCB design/WPS_Scaled/sensors.kicad_sch (KiCad schematic)
At the start: 26 parts, among them J10 KF350-3.5-3P, J11 KF350-3.5-3P, J12-A KF350-3.5-2P, J12-B KF350-3.5-2P, J12-C KF350-3.5-2P, J5 KF350-3.5-3P, J6 KF350-3.5-3P, J7 KF350-3.5-3P, J8-A KF350-3.5-2P, J8-B KF350-3.5-2P, J9-A KF350-3.5-2P, J9-B KF350-3.5-2P

Commit message: finalized the pcb schematics
Parts:
- added R29, R30, R31, R32: 4.7k, symbol Device:R
- renumbered J12-A to J12-A1, J12-B to J12-B1, J12-C to J12-C1, J8-A to J8-A1, J8-B to J8-B1, J9-A to J9-A1, J9-B to J9-B1, R3 to R15, R4 to R16
Connections:
- net GND is gone; now on net +3.3V: C15.2, C16.2, C17.2, C18.2, J10.3, J11.3, J12-A1.2, J5.3, J6.3, J7.3, J8-B1.1, J9-B1.2, R12.2, R14.2, R16.2, R18.2
- net +3.3V: now also R29.2, R30.2, R31.2, R32.2
- net SENSOR_COLOR_SCL: now also R30.1
- net SENSOR_COLOR_SDA: now also R29.1
- net SENSOR_CURRENT_SCL: now also R31.1
- net SENSOR_CURRENT_SDA: now also R32.1
Other:
- note added: "Current and Voltage sensor (INA219)"
- note removed: "Water Current sensor (INA219)"
- company: (none) -> Makerere University
- moved on the sheet: J12-A1, J12-B1, J12-C1, J8-A1, J8-B1, R18

Commit message: finallized pcb layout
Parts:
- removed R29, R30, R31, R32: 4.7k, symbol Device:R
- C15, C16, C17, C18: footprint (none) -> COIL:CAP-TH_L3.6-W2.3-P2.50-D0.5
- J10, J11, J5, J6, J7: footprint :CONN-TH_3P-P3.50_KF350-3.5-3P -> COIL:CONN-TH_3P-P3.50_KF350-3.5-3P
- J12-A1, J12-B1, J12-C1, J8-A1, J8-B1, J9-A1, J9-B1: footprint :CONN-TH_P3.50_KF350-3.5-2P -> COIL:CONN-TH_P3.50_KF350-3.5-2P
- R11, R12, R13, R14, R15, R16, R17, R18, R19, R20: footprint (none) -> COIL:RES-TH_BD2.4-L6.3-P10.30-D0.6
Connections:
- net PRE_SIG: now reaches J6.1, R13.1
- net TURB_SIG: now reaches J5.1, R11.1
- net PH_SIG: now reaches J11.1, R20.1
- net TDS_SIG: now reaches J10.1, R19.1
- net FLOW_SIG: now reaches J7.1, R15.1
- net LEV_ECHO: now reaches J9-B1.1, R17.1
- net +3.3V renamed GND
- net GND: no longer J12-A1.1, J8-B1.2
- new net +3V3: J12-A1.1, J8-B1.2
Other:
- moved on the sheet: J12-A1, J12-B1, J12-C1, J9-A1, J9-B1, R17, R18
