File: hardware/PCB design/WPS_Scaled/WPS_Scaled.kicad_pcb (KiCad board)
At the start: 4 copper layers, 141.5 x 107 mm, 119 parts, among them J1 KF128-5.08-2P, J10 KF350-3.5-3P, J11 KF350-3.5-3P, J12-A1 KF350-3.5-2P, J12-B1 KF350-3.5-2P, J12-C1 KF350-3.5-2P, J13 ZX-XH2.54-2PZZ, J14 2.54-1*4P母, J15 ZX-XH2.54-2PZZ, J16 ZX-XH2.54-2PZZ, J2 KF128-5.08-2P, J3 KF128-5.08-2P, J4 KF128-5.08-2P, J5 KF350-3.5-3P, J6 KF350-3.5-3P, J7 KF350-3.5-3P, J8-A1 KF350-3.5-2P, J8-B1 KF350-3.5-2P, J9-A1 KF350-3.5-2P, J9-B1 KF350-3.5-2P, K1 SRD-05VDC-SL-C, K2 SRD-05VDC-SL-C, K3 SRD-05VDC-SL-C, Q1 2N2222, Q2 IRF9540NPBF, Q3 2N2222, Q4 2N2222, Q5 2N2222, U1 LM2595T-5.0, U2 TLV1117LV33DCYR, U3 ESP32-S3-WROOM-1(N16R8), U4 TYPEC-306DDW-ARP16, U5 CH340C

Commit message: updated the pcb component placements
Parts:
- added H1: MountingHole, MountingHole:MountingHole_3.2mm_M3, F.Cu at (78.7, 53.3)
- added H2: MountingHole, MountingHole:MountingHole_3.2mm_M3, F.Cu at (78.7, 152.4)
- added H3: MountingHole, MountingHole:MountingHole_3.2mm_M3, F.Cu at (186.7, 153.7)
- added H4: MountingHole, MountingHole:MountingHole_3.2mm_M3, F.Cu at (185.4, 53.3)
- moved TP1 189.2 mm to (-11.6, 20.0)
- moved TP2 189.2 mm to (-11.5, 26.1)
- moved TP5 167.9 mm to (-47.0, 24.1)
- moved TP3 166.1 mm to (-22.7, 23.8)
- moved NT1 162.8 mm to (-30.5, 61.5)
- moved TP4 162.8 mm to (-51.7, 50.7)
- moved LED1 141.8 mm to (185.5, 125.8), turned to 180 degrees
- moved LED2 135.8 mm to (185.5, 132.1), turned to 180 degrees
- moved R7 133.2 mm to (171.6, 128.3), turned to 0 degrees
- moved LED3 130.2 mm to (185.5, 138.4), turned to 180 degrees
- moved J4 127.7 mm to (183.7, 114.3), turned to 90 degrees
- moved D9 127.4 mm to (172.3, 109.2)
- moved J5 126.6 mm to (176.3, 153.7), turned to 0 degrees
- moved R26 126.6 mm to (171.6, 132.4), turned to 0 degrees
- moved LED4 126.4 mm to (185.5, 144.8), turned to 180 degrees
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Other:
- board size 141.5 x 107 mm -> 115 x 108 mm
- copper layers 4 -> 2

Commit message: finalized the pcb component placement for version 2
Parts:
- moved TP5 201.7 mm to (130.8, 119.4)
- moved TP2 192.2 mm to (176.5, 66.0)
- moved TP1 188.7 mm to (171.4, 66.0)
- moved NT1 174.8 mm to (141.5, 92.7), turned to 180 degrees
- moved TP4 174.0 mm to (113.0, 106.7)
- moved TP11 172.5 mm to (106.7, 109.2)
- moved TP10 168.7 mm to (106.7, 104.1)
- moved TP3 168.6 mm to (133.3, 87.6)
- moved TP9 157.4 mm to (105.4, 61.0)
- moved TP8 134.9 mm to (96.5, 82.5)
- moved TP7 132.3 mm to (96.5, 78.7)
- moved TP6 106.3 mm to (91.4, 61.0)
- moved LED1 68.7 mm to (116.8, 127.0), turned to -90 degrees
- moved LED2 62.5 mm to (123.2, 127.0), turned to -90 degrees
- moved LED3 57.1 mm to (129.5, 127.0), turned to -90 degrees
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Other:
- board size 115 x 108 mm -> 120 x 115 mm

Commit message: started routing with sensors and critical signals
Parts:
- moved J16 100.3 mm to (88.9, 55.9)
- moved J15 87.9 mm to (97.8, 54.6), turned to 0 degrees
- moved R24 76.2 mm to (109.2, 69.8), turned to -90 degrees
- moved R25 73.8 mm to (104.1, 69.8), turned to -90 degrees
- moved TP4 49.7 mm to (64.1, 115.6)
- moved R14 45.7 mm to (110.5, 144.8)
- moved R13 45.7 mm to (105.4, 144.8)
- moved TP10 43.8 mm to (62.9, 104.8)
- moved TP11 43.8 mm to (62.9, 109.9)
- moved R32 40.6 mm to (123.2, 144.1), turned to -90 degrees
- moved R33 40.6 mm to (119.4, 144.1), turned to 90 degrees
- moved R12 40.6 mm to (138.4, 144.1)
- moved R20 40.6 mm to (130.8, 144.1)
- moved R11 40.6 mm to (134.6, 144.1)
- moved R19 40.6 mm to (127.0, 144.1)
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Connections:
- Q3 pad 1: GNDPWR -> GND
- Q4 pad 1: GNDPWR -> GND
- Q5 pad 1: GNDPWR -> GND
- U3 pad 10: /Actuators/ACTUATOR_VALVE_EN -> unconnected-(U3-IO17-Pad10)
- U3 pad 11: /ESP32_Module/LED_POWER_ON -> unconnected-(U3-IO18-Pad11)
- U3 pad 12: /ESP32_Module/LED_MAINTENANCE -> unconnected-(U3-IO8-Pad12)
- U3 pad 30: unconnected-(U3-IO37-Pad30) -> /ESP32_Module/LED_MAINTENANCE
- U3 pad 31: unconnected-(U3-IO38-Pad31) -> /ESP32_Module/LED_POWER_ON
- U3 pad 32: unconnected-(U3-IO39-Pad32) -> /Actuators/ACTUATOR_VALVE_EN
- U3 pad 33: unconnected-(U3-IO40-Pad33) -> /Actuators/ACTUATOR_UV_EN
- U3 pad 34: unconnected-(U3-IO41-Pad34) -> /Actuators/ACTUATOR_PUMP_EN
- U3 pad 8: /Actuators/ACTUATOR_PUMP_EN -> unconnected-(U3-IO15-Pad8)
- U3 pad 9: /Actuators/ACTUATOR_UV_EN -> unconnected-(U3-IO16-Pad9)
Routing:
- net /ESP32_Module/I2C1_SDA: track 0.00 -> 164.2 mm, vias 0 -> 2
- net /ESP32_Module/I2C1_SCL: track 0.00 -> 144.9 mm, vias 0 -> 2
- net /ESP32_Module/BUTTON_EN: track 0.00 -> 125.4 mm, vias 0 -> 2
- net /ESP32_Module/SENSOR_TURBIDITY_SIGNAL: track 0.00 -> 85.3 mm, vias 0 -> 2
- net /ESP32_Module/BUTTON_SYSTEM_RESET: track 0.00 -> 74.9 mm, vias 0 -> 2
- net /ESP32_Module/SENSOR_PH_SIGNAL: track 0.00 -> 73.8 mm, vias 0 -> 1
- net /ESP32_Module/I2C2_SCL: track 0.00 -> 65.6 mm, vias 0 -> 2
- net /ESP32_Module/SENSOR_TDS_SIGNAL: track 0.00 -> 65.2 mm, vias 0 -> 1
- net /ESP32_Module/I2C2_SDA: track 0.00 -> 59.9 mm, vias 0 -> 2
- net /ESP32_Module/USB_DP: track 0.00 -> 48.4 mm
- net /ESP32_Module/USB_DN: track 0.00 -> 48.4 mm
- net /ESP32_Module/SENSOR_PRESSURE_SIGNAL: track 0.00 -> 44.3 mm, vias 0 -> 1
- net /ESP32_Module/SENSOR_FLOW_SIGNAL: track 0.00 -> 36.7 mm, vias 0 -> 1
- net /ESP32_Module/UART_RX: track 0.00 -> 35.9 mm, vias 0 -> 2
- net /ESP32_Module/UART_TX: track 0.00 -> 35.5 mm, vias 0 -> 2
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- added copper zone on In1.Cu, net GND
- added copper zone on In2.Cu, net GND
- added copper zone on In1.Cu, net GNDPWR
- added copper zone on In2.Cu, net GNDPWR
Other:
- copper layers 2 -> 4

Commit message: continued with routing the pcb
Parts:
- moved R5 74.4 mm to (112.1, 69.8)
- moved TP5 70.0 mm to (61.0, 124.5)
- moved C1 64.3 mm to (172.7, 57.8), turned to 90 degrees
- moved TP3 50.2 mm to (151.1, 40.6)
- moved C2 48.7 mm to (161.9, 57.8), turned to 90 degrees
- moved R26 47.2 mm to (127.7, 130.0)
- moved R27 47.2 mm to (132.5, 130.1)
- moved R28 47.2 mm to (136.3, 130.0)
- moved R7 47.2 mm to (123.6, 130.0)
- moved LED1 45.6 mm to (122.4, 121.0)
- moved LED2 45.6 mm to (128.8, 121.0)
- moved LED3 45.6 mm to (135.1, 121.0)
- moved LED4 45.6 mm to (141.5, 121.0)
- moved TP1 34.3 mm to (212.1, 68.6)
- moved TP2 34.3 mm to (212.1, 63.5)
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Routing:
- net +5V: track 0.00 -> 291.1 mm, vias 0 -> 4
- net +5V_SW: track 0.00 -> 285.2 mm, vias 0 -> 3
- net VBAT: track 0.00 -> 261.1 mm, vias 0 -> 3
- net +3V3: track 6.42 -> 267.3 mm, vias 0 -> 5
- net /Actuators/ACTUATOR_PUMP_EN: track 0.00 -> 137.1 mm, vias 0 -> 2
- net /Power_Management/VBAT_PROTECTED: track 0.00 -> 137.0 mm, vias 0 -> 1
- net /Actuators/ACTUATOR_UV_EN: track 0.00 -> 98.7 mm, vias 0 -> 2
- net /Actuators/ACTUATOR_VALVE_EN: track 0.00 -> 73.1 mm, vias 0 -> 2
- net GNDPWR: track 0.00 -> 63.3 mm, vias 0 -> 2
- net /Power_Management/BUCK_FB: track 0.00 -> 47.0 mm, vias 0 -> 1
- net /Actuators/RELAY3_COIL: track 0.00 -> 44.8 mm
- net /Actuators/RELAY2_COIL: track 0.00 -> 44.3 mm
- net /Actuators/RELAY1_COIL: track 0.00 -> 43.0 mm
- net /ESP32_Module/BUTTON_BOOT: track 28.9 -> 63.9 mm
- net /Power_Management/BUCK_OUT: track 0.00 -> 31.5 mm
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