File: hardware/PCB design/WPS_Scaled/_autosave-Power_Management.kicad_sch (KiCad schematic)
At the start: 25 parts, among them J1 KF128-5.08-2P, Q1 2N2222, Q2 IRF9540NPBF, U1 LM2595T-5.0, U2 TLV1117LV33DCYR

Commit message: finalized the routing
Parts:
- TP12: footprint (none) -> TestPoint:TestPoint_THTPad_D2.0mm_Drill1.0mm
Changed lines of the file:
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@@
 			)
 		)
-		(property "Footprint" ""
+		(property "Footprint" "TestPoint:TestPoint_THTPad_D2.0mm_Drill1.0mm"
 			(at 217.17 55.88 0)
 			(effects
